File: sensor-v2-board/sensor-v2-board/sensor-v2-board.sch (KiCad schematic (older format))
At the start: 56 parts, among them J1 Conn_01x03_Male, J2 Conn_01x03_Male, J3 Conn_01x03_Male, J4 Conn_01x02_Male, J5 Conn_01x04_Male, J6 Conn_01x04_Male, J7 Conn_01x05_Male, J8 USB_B_Micro, SW1 RST_Push, SW2 Boot_Switch, U1 NCP1117-3.3_SOT223, U2 SN65HVD232, U3 STM32F042K6Tx, U4 FT230XQ, Y1 8MHz

Commit message: new PCB for 2022
Parts:
- J8: symbol Connector:USB_B_Micro -> sensor-v2-board-rescue:USB_B_Micro-Connector
Changed lines of the file:
@@
 $EndComp
 $Comp
-L Connector:USB_B_Micro J8
+L sensor-v2-board-rescue:USB_B_Micro-Connector J8
 U 1 1 60CFC842
 P 9250 2800
