File: PCB_Principal_V2/Carte Principale.kicad_pcb (KiCad board)
At the start: 2 copper layers, 80 x 65 mm, 44 parts, among them IC2 SN65HVD232D, J1 MOLEX_4DROIT, J10 22-?-0527-2051, J11 22-?-0527-2051, J13 62000411622, J2 MOLEX_4DROIT, J3 MOLEX_3DROIT, J4 MOLEX_3DROIT, J5 MOLEX_3DROIT, J6 645002117322, J7 Serial extern, J9 62000411622

Commit message: ajout v3 carte alim
Routing:
- net /S2_D: track 26.8 -> 27.9 mm
- net /S3_D: track 23.2 -> 24.3 mm
- net /CANL: track 41.5 -> 42.5 mm
- net GND: vias 7 -> 27
Other:
- board text added: "3V3"
- board text added: "GND"
- board text added: "RX"
- board text added: "TX"

Commit message: some changes
Other:
- board text removed: "CAN + 5VC"
