File: PCB_Pompe_V2/PCB_Pompe_V2.sch (KiCad schematic (older format))
At the start: 129 parts, among them J1 Conn_01x04_Female, J10 Conn_01x03_Female, J11 Conn_01x03_Female, J12 Conn_01x03_Female, J13 Conn_01x05_Female, J2 Conn_01x04_Female, J3 Conn_01x03_Female, J4 Conn_01x03_Female, J5 Conn_01x03_Female, J6 Conn_01x03_Female, J7 Conn_01x03_Female, J8 Conn_01x02_Male, J9 Conn_01x03_Female, Q1 DMN10H700S, Q10 DMN10H700S, Q11 DMN10H700S, Q12 DMN10H700S, Q13 DMN10H700S, Q14 DMN10H700S, Q15 DMN10H700S, Q16 DMN10H700S, Q17 DMN10H700S, Q18 DMN10H700S, Q2 DMN10H700S, Q3 DMN10H700S, Q4 DMN10H700S, Q5 DMN10H700S, Q6 DMN10H700S, Q7 DMN10H700S, Q8 DMN10H700S, Q9 DMN10H700S, U1 SN65HVD232, U2 STM32F042K6Tx, U3 MCP1703A-3002_SOT23, Y1 8MHz

Commit message: add MM connector + modification schematic pcb pump+ final routing IO
Parts:
- removed D10, D11, D12, D13, D14, D15, D16, D17, D18, D19, D20, D3, D4, D5, D6, D7, D8, D9: D, Diode_SMD:D_SOD-323, symbol Device:D
- removed J10, J11, J12, J3, J4, J5, J6, J7, J9: Conn_01x03_Female, AREA_lib_Connector:Wuerth_2mm_3pin62000311622, symbol Connector:Conn_01x03_Female
- removed Q1, Q10, Q11, Q12, Q13, Q14, Q15, Q16, Q17, Q18, Q2, Q3, Q4, Q5, Q6, Q7, Q8, Q9: DMN10H700S, Package_TO_SOT_SMD:SOT-23, symbol Transistor_FET:DMN10H700S
- removed R14, R15, R16, R17, R18, R19, R20: 10k, Resistor_SMD:R_0603_1608Metric_Pad0.98x0.95mm_HandSolder, symbol Device:R
- removed U2: STM32F042K6Tx, Package_QFP:LQFP-32_7x7mm_P0.8mm, symbol MCU_ST_STM32F0:STM32F042K6Tx
- removed U3: MCP1703A-3002_SOT23, Package_TO_SOT_SMD:SOT-23, symbol Regulator_Linear:MCP1703A-3002_SOT23
- added C13, C14: 100nF, Capacitor_SMD:C_0805_2012Metric_Pad1.18x1.45mm_HandSolder, symbol Device:C
- added D10, D11, D12, D13, D14, D3, D4, D5, D6, D7, D8, D9: LED_DEBUG, LED_SMD:LED_0805_2012Metric_Pad1.15x1.40mm_HandSolder, symbol Device:LED
- added H1, H2, H3, H4: MountingHole_Pad, MountingHole:MountingHole_3.2mm_M3_Pad_Via, symbol Mechanical:MountingHole_Pad
- added SW1: SW_Push, Button_Switch_SMD:SW_SPST_FSMSM, symbol Switch:SW_Push
- added U2: STM32F302C6Tx, Package_QFP:LQFP-48_7x7mm_P0.5mm, symbol MCU_ST_STM32F3:STM32F302C6Tx
- added U?: NCP1117-3.3_SOT223, Package_TO_SOT_SMD:SOT-223-3_TabPin2, symbol Regulator_Linear:NCP1117-3.3_SOT223
- C1, C2, C3, C4, C5, C7: footprint Capacitor_SMD:C_0603_1608Metric_Pad1.08x0.95mm_HandSolder -> Capacitor_SMD:C_0805_2012Metric_Pad1.18x1.45mm_HandSolder
- C6: value 10µF -> 1u; footprint Capacitor_SMD:C_0603_1608Metric_Pad1.08x0.95mm_HandSolder -> Capacitor_SMD:C_0805_2012Metric_Pad1.18x1.45mm_HandSolder
- C8, C9: value 1µF -> 10u; footprint Capacitor_SMD:C_0603_1608Metric_Pad1.08x0.95mm_HandSolder -> Capacitor_SMD:C_0805_2012Metric_Pad1.18x1.45mm_HandSolder
- D1, D21, D22, D23, D24, D25, D26, D27, D28, D29, D30, D31, D32, D33, D34, D35, D36, D37, D38, D39, D40: footprint LED_SMD:LED_0603_1608Metric_Pad1.05x0.95mm_HandSolder -> LED_SMD:LED_0805_2012Metric_Pad1.15x1.40mm_HandSolder
- J1, J2: footprint AREA_lib_Connector:Wuerth_2mm_4pin_62000411622 -> AREA_lib_Connector:690367290476
- R1, R10, R11, R12, R13, R3, R4, R5, R6, R7, R8, R9: value 10k -> 560; footprint Resistor_SMD:R_0603_1608Metric_Pad0.98x0.95mm_HandSolder -> Resistor_SMD:R_0805_2012Metric_Pad1.20x1.40mm_HandSolder
- R2, R21, R22, R23, R24, R25, R26, R27, R28, R29, R30, R31, R32, R33, R34, R35, R36, R37, R38, R39, R40, R41: footprint Resistor_SMD:R_0603_1608Metric_Pad0.98x0.95mm_HandSolder -> Resistor_SMD:R_0805_2012Metric_Pad1.20x1.40mm_HandSolder
Connections:
- net labels added: BOOT, OUT_P10, OUT_P11, OUT_P12, OUT_P13, OUT_P14, OUT_P15, OUT_V10, OUT_V11, OUT_V13, OUT_V14, OUT_V15, P10, P11, P12, P13, P14, P15, V10, V11, V12, V13, V14, V15
- wire segments 106 -> 76
- no-connect marks 0 -> 1
Other:
- moved on the sheet: C1, C10, C11, C12, C2, C3, C4, C5, C7, C8, C9, D1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

Commit message: add pcb esp32 + changes on pump pcb
Parts:
- removed C11, C12: 100µF, Capacitor_THT:CP_Radial_D10.0mm_P3.80mm, symbol Device:CP
- removed D10, D11, D12, D13, D14, D23, D24, D25, D26, D27, D28, D29, D3, D30, D31, D32, D33, D34, D35, D36, D37, D38, D39, D4, D40, D5, D6, D7, D8, D9: LED_DEBUG, LED_SMD:LED_0805_2012Metric_Pad1.15x1.40mm_HandSolder, symbol Device:LED
- removed R1, R10, R11, R12, R13, R24, R25, R26, R27, R28, R29, R3, R30, R31, R32, R33, R34, R35, R36, R37, R38, R39, R4, R40, R41, R5, R6, R7, R8, R9: 560, Resistor_SMD:R_0805_2012Metric_Pad1.20x1.40mm_HandSolder, symbol Device:R
- gave numbers to parts that had none: 1
Connections:
- net labels removed: OUT_P1, OUT_P10, OUT_P11, OUT_P12, OUT_P13, OUT_P14, OUT_P15, OUT_P2, OUT_P3, OUT_P4, OUT_P5, OUT_P6, OUT_P7, OUT_P8, OUT_P9, OUT_V1, OUT_V10, OUT_V11, OUT_V13, OUT_V14, OUT_V15, OUT_V2, OUT_V3, OUT_V4, OUT_V5, OUT_V6, OUT_V7, OUT_V8, OUT_V9
- wire segments 76 -> 41
