File: IO_Board_V1/IO_Board_V1.sch (KiCad schematic (older format))
At the start: 92 parts, among them J1 USB_C_Receptacle_USB2.0, J10 IFM1, J11 FOURCHE, J12 BTN, J13 FOURCHE, J14 BTN, J15 CON_UART, J16 BTN, J17 FOURCHE, J18 IFM2, J19 IFM3, J2 CON_debug, J20 FOURCHE, J21 CON_I2C, J22 IFM4, J23 SPI, J24 BTN, J3 Conn_ARM_JTAG_SWD_10, J4 CON_CAN, J5 CON_CAN, J6 12V, J7 BTN, J8 BTN, J9 IFM0, SW1 BOOT, SW2 RST, U1 STM32F302C6Tx, U2 NCP1117-3.3_SOT223, U3 SN65HVD232, Y1 8MHz

Commit message: change connector and some final touch
Parts:
- J4, J5: footprint AREA_lib_Connector:Wuerth_2mm_4pin_62000411622 -> AREA_lib_Connector:690367290476
Changed lines of the file:
@@
 F 0 "J4" H 8800 2950 50  0000 C CNN
 F 1 "CON_CAN" H 8650 2800 50  0000 C CNN
-F 2 "AREA_lib_Connector:Wuerth_2mm_4pin_62000411622" H 8850 2850 50  0001 C CNN
+F 2 "AREA_lib_Connector:690367290476" H 8850 2850 50  0001 C CNN
 F 3 "~" H 8850 2850 50  0001 C CNN
 	1    8850 2850
@@
 F 0 "J5" H 10050 2950 50  0000 C CNN
 F 1 "CON_CAN" H 9900 2800 50  0000 C CNN
-F 2 "AREA_lib_Connector:Wuerth_2mm_4pin_62000411622" H 10100 2850 50  0001 C CNN
+F 2 "AREA_lib_Connector:690367290476" H 10100 2850 50  0001 C CNN
 F 3 "~" H 10100 2850 50  0001 C CNN
 	1    10100 2850
