File: Rmeasure_V1_Board/Rmeasure_V1_Board.sch (KiCad schematic (older format))
At the start: 52 parts, among them J1 USB_C_Receptacle_USB2.0, J2 CON_debug, J3 Conn_ARM_JTAG_SWD_10, J4 CON_CAN, J5 CON_CAN, SW1 BOOT, SW2 RST, U1 STM32F302C6Tx, U2 NCP1117-3.3_SOT223, U3 SN65HVD232, Y1 8MHz

Commit message: change rgb on rmeasure + add library component
Parts:
- removed D4: LED_RGBA, LED_SMD:LED_SK6812_EC15_1.5x1.5mm, symbol Device:LED_RGBA
- added D4: LED_RGB, AREA_lib_composant:LED_RGB_LTRBRASF6B6C011200R18, symbol Device:LED_RGB
- J1: symbol Connector:USB_C_Receptacle_USB2.0 -> Rmeasure_V1_Board-rescue:USB_C_Receptacle_USB2.0-Connector
- J2: footprint AREA_lib_Connector:Wuerth_2mm_4pin_62000411622 -> AREA_lib_Connector:Wuerth_2.54mm_4pins_61900411121
- J4, J5: footprint AREA_lib_Connector:Wuerth_2mm_4pin_62000411622 -> AREA_lib_Connector:690367290476
Connections:
- net GND: now also D4.4 (BA), D4.5 (GA), D4.6 (RA)
- net at R5.1: now also D4.1 (RK)
- net at R6.1: now also D4.2 (GK)
- net at R7.1: now also D4.3 (BK)
Changed lines of the file:
@@
 F 0 "J4" H 7600 4850 50  0000 C CNN
 F 1 "CON_CAN" H 7450 4700 50  0000 C CNN
-F 2 "AREA_lib_Connector:Wuerth_2mm_4pin_62000411622" H 7650 4750 50  0001 C CNN
+F 2 "AREA_lib_Connector:690367290476" H 7650 4750 50  0001 C CNN
 F 3 "~" H 7650 4750 50  0001 C CNN
 	1    7650 4750
@@
 F 0 "J5" H 8850 4850 50  0000 C CNN
 F 1 "CON_CAN" H 8700 4700 50  0000 C CNN
-F 2 "AREA_lib_Connector:Wuerth_2mm_4pin_62000411622" H 8900 4750 50  0001 C CNN
+F 2 "AREA_lib_Connector:690367290476" H 8900 4750 50  0001 C CNN
 F 3 "~" H 8900 4750 50  0001 C CNN
 	1    8900 4750
@@
 Bleu
 Wire Wire Line
-	4400 7150 4600 7150
-$Comp
-L Device:LED_RGBA D4
-U 1 1 61698EB2
-P 4200 7150
-F 0 "D4" H 4200 7647 50  0000 C CNN
-F 1 "LED_RGBA" H 4200 7556 50  0000 C CNN
-F 2 "LED_SMD:LED_SK6812_EC15_1.5x1.5mm" H 4200 7100 50  0001 C CNN
-F 3 "~" H 4200 7100 50  0001 C CNN
-	1    4200 7150
-	1    0    0    -1
-$EndComp
-$Comp
-L power:+3.3V #PWR023
-U 1 1 61699C32
-P 4600 7150
-F 0 "#PWR023" H 4600 7000 50  0001 C CNN
-F 1 "+3.3V" H 4600 7300 50  0000 C CNN
-F 2 "" H 4600 7150 50  0001 C CNN
-F 3 "" H 4600 7150 50  0001 C CNN
-	1    4600 7150
-	1    0    0    -1
-$EndComp
+	4500 7150 4700 7150
 Wire Wire Line
 	9200 1300 9450 1300
@@
 F 0 "J2" H 5050 1000 50  0000 C CNN
 F 1 "CON_debug" H 4900 850 50  0000 C CNN
-F 2 "AREA_lib_Connector:Wuerth_2mm_4pin_62000411622" H 5100 900 50  0001 C CNN
+F 2 "AREA_lib_Connector:Wuerth_2.54mm_4pins_61900411121" H 5100 900 50  0001 C CNN
 F 3 "~" H 5100 900 50  0001 C CNN
 	1    5100 900
@@
 	5850 7000 5600 7000
 $Comp
-L Connector:USB_C_Receptacle_USB2.0 J1
+L Rmeasure_V1_Board-rescue:USB_C_Receptacle_USB2.0-Connector J1
 U 1 1 61685184
 P 5150 2000
@@
 NoConn ~ 3150 5500
 NoConn ~ 3150 6200
+$Comp
+L Device:LED_RGB D4
+U 1 1 6180651B
+P 4200 7150
+F 0 "D4" H 4200 7647 50  0000 C CNN
+F 1 "LED_RGB" H 4200 7556 50  0000 C CNN
+F 2 "AREA_lib_composant:LED_RGB_LTRBRASF6B6C011200R18" H 4200 7100 50  0001 C CNN
+F 3 "~" H 4200 7100 50  0001 C CNN
+	1    4200 7150
+	1    0    0    -1
+$EndComp
+Wire Wire Line
+	4400 6950 4500 6950
+Wire Wire Line
+	4500 6950 4500 7150
+Wire Wire Line
+	4500 7150 4500 7350
+Wire Wire Line
+	4500 7350 4400 7350
+Connection ~ 4500 7150
+Wire Wire Line
+	4400 7150 4500 7150
+$Comp
+L power:GND #PWR0101
+U 1 1 6185EE35
+P 4700 7150
+F 0 "#PWR0101" H 4700 6900 50  0001 C CNN
+F 1 "GND" H 4705 6977 50  0000 C CNN
+F 2 "" H 4700 7150 50  0001 C CNN
+F 3 "" H 4700 7150 50  0001 C CNN
+	1    4700 7150
+	1    0    0    -1
+$EndComp
 $EndSCHEMATC
